File: cnc_adapter/cnc_adapter.kicad_sch (KiCad schematic)
At the start: 12 parts, among them J1 DB25_Plug, J2 Conn_01x15_Socket, J3 Conn_01x15_Socket

Commit message: Finish draft
Parts:
- added H1, H2, H3, H4: MountingHole, MountingHole:MountingHole_2.7mm_M2.5, symbol Mechanical:MountingHole
- C1, C2, C3, C4: footprint (none) -> Capacitor_SMD:C_0603_1608Metric
