File: cnc_adapter/cnc_adapter.kicad_pcb (KiCad board)
At the start: 2 copper layers, 50.2 x 40.7 mm, 8 parts, among them J1 DB25_Plug, J2 Conn_01x15_Socket, J3 Conn_01x15_Socket

Commit message: Finish draft
Parts:
- added C1: 100nF, Capacitor_SMD:C_0603_1608Metric, F.Cu at (85.8, 77.0)
- added C2: 100nF, Capacitor_SMD:C_0603_1608Metric, F.Cu at (85.8, 79.0)
- added C3: 100nF, Capacitor_SMD:C_0603_1608Metric, F.Cu at (85.8, 81.3)
- added C4: 100nF, Capacitor_SMD:C_0603_1608Metric, F.Cu at (85.8, 83.3)
- added H1: MountingHole, MountingHole:MountingHole_2.7mm_M2.5, F.Cu at (45.7, 51.5)
- added H2: MountingHole, MountingHole:MountingHole_2.7mm_M2.5, F.Cu at (45.7, 87.1)
- added H3: MountingHole, MountingHole:MountingHole_2.7mm_M2.5, F.Cu at (84.8, 51.5)
- added H4: MountingHole, MountingHole:MountingHole_2.7mm_M2.5, F.Cu at (84.8, 87.1)
Routing:
- net D26: track 44.4 -> 42.4 mm
- net D34: track 45.4 -> 47.1 mm
- net D35: track 46.8 -> 48.5 mm
- net D19: track 31.2 -> 32.6 mm
- net D32: track 46.8 -> 48.2 mm
- net D33: track 44.7 -> 44.0 mm

Commit message: Add version silkscreen
Other:
- board text added: "2025.06.04"
- board text added: "PopLab CNC Adapter v0.1"
- board text added: "https://github.com/nebularnoise/PopLab_CNC"
Changed lines of the file:
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@@
 		(layer "Edge.Cuts")
+	)
+	(gr_text "https://github.com/nebularnoise/PopLab_CNC"
+		(at 85.344 72.136 0)
+		(layer "B.SilkS")
+		(effects
+			(font
+				(size 1 1)
+				(thickness 0.1)
+			)
+			(justify left bottom mirror)
+		)
+	)
+	(gr_text "2025.06.04"
+		(at 60.452 77.724 0)
+		(layer "B.SilkS")
+		(effects
+			(font
+				(size 1 1)
+				(thickness 0.1)
+			)
+			(justify left bottom mirror)
+		)
+	)
+	(gr_text "PopLab CNC Adapter v0.1"
+		(at 80.772 66.294 0)
+		(layer "B.SilkS")
+		(effects
+			(font
+				(size 1 1)
+				(thickness 0.1)
+			)
+			(justify left bottom mirror)
+		)
 	)
 	(dimension
